Commit message: Refactor Xense camera configuration and update URDF mass value. Adjusted default rectify_size and output type handling in XenseTactileCamera. Updated gripper_open_readout values and modified dataset parameters in bi_arx5 documentation.

File: src/lerobot/robots/bi_arx5/ARX5_SDK/models/X5.urdf (robot description, URDF)
Before this commit: robot X5, 8 links, 7 joints
Links:
- link link6: mass 0.65 -> 0.7
